File: Hardware/Thruster-Commander.sch (EAGLE design)
At the start: 27 parts, among them U5 MC7805, Y1 8Mhz

Commit message: rev3 version.
Connections:
- removed net PWM2: AVR_ICSP.1
- net +5V: now also IN_EXT0.3, IN_EXT1.3; no longer IN_EXT0.2, IN_EXT1.2
- net GND: now also LED2.C, LED3.C; no longer R5.1, R6.1
- net INPUT_EXT0: now also IN_EXT0.2; no longer IN_EXT0.3
- net INPUT_EXT1: now also IN_EXT1.2; no longer IN_EXT1.3
- net INPUT_INT: no longer AVR_ICSP.3
- net LED_EXT0: now also R5.2; no longer LED2.A
- net LED_EXT1: now also R6.2; no longer LED3.A
- net LED_INT: now also AVR_ICSP.3
- net N$2: now also LED2.A, R5.1; no longer LED2.C, R5.2
- net N$5: now also LED3.A, R6.1; no longer LED3.C, R6.2
- net PWM0: now also AVR_ICSP.4
- net PWM1: now also AVR_ICSP.1; no longer AVR_ICSP.4
Other:
- moved on the sheet: LED2, LED3, R5, R6
Changed lines of the file:
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@@
 <instance part="Y1" gate="G$1" x="114.3" y="119.38" rot="R90"/>
 <instance part="GND6" gate="1" x="127" y="114.3"/>
-<instance part="LED2" gate="G$1" x="60.96" y="38.1"/>
-<instance part="R5" gate="G$1" x="60.96" y="25.4" rot="R90"/>
+<instance part="LED2" gate="G$1" x="60.96" y="25.4"/>
+<instance part="R5" gate="G$1" x="60.96" y="35.56" rot="R90"/>
 <instance part="GND1" gate="1" x="60.96" y="15.24"/>
-<instance part="LED3" gate="G$1" x="76.2" y="38.1"/>
-<instance part="R6" gate="G$1" x="76.2" y="25.4" rot="R90"/>
+<instance part="LED3" gate="G$1" x="76.2" y="25.4"/>
+<instance part="R6" gate="G$1" x="76.2" y="35.56" rot="R90"/>
 <instance part="GND7" gate="1" x="76.2" y="15.24"/>
 <instance part="C4" gate="G$1" x="78.74" y="160.02"/>
@@
 </segment>
 <segment>
+<pinref part="LED2" gate="G$1" pin="C"/>
 <pinref part="GND1" gate="1" pin="GND"/>
-<pinref part="R5" gate="G$1" pin="1"/>
-<wire x1="60.96" y1="17.78" x2="60.96" y2="20.32" width="0.1524" layer="91"/>
+<wire x1="60.96" y1="20.32" x2="60.96" y2="17.78" width="0.1524" layer="91"/>
 </segment>
 <segment>
 <pinref part="GND7" gate="1" pin="GND"/>
-<pinref part="R6" gate="G$1" pin="1"/>
+<pinref part="LED3" gate="G$1" pin="C"/>
 <wire x1="76.2" y1="17.78" x2="76.2" y2="20.32" width="0.1524" layer="91"/>
 </segment>
@@
 </segment>
 <segment>
-<pinref part="IN_EXT0" gate="G$1" pin="2"/>
-<wire x1="177.8" y1="144.78" x2="187.96" y2="144.78" width="0.1524" layer="91"/>
-<label x="187.96" y="144.78" size="1.778" layer="95" rot="MR0"/>
-</segment>
-<segment>
-<wire x1="215.9" y1="144.78" x2="226.06" y2="144.78" width="0.1524" layer="91"/>
-<pinref part="IN_EXT1" gate="G$1" pin="2"/>
-<label x="226.06" y="144.78" size="1.778" layer="95" rot="MR0"/>
-</segment>
-<segment>
 <pinref part="C3" gate="G$1" pin="1"/>
 <wire x1="25.4" y1="35.56" x2="25.4" y2="48.26" width="0.1524" layer="91"/>
@@
 <label x="114.3" y="142.24" size="1.778" layer="95"/>
 </segment>
-</net>
-<net name="PWM2" class="0">
-<segment>
-<pinref part="AVR_ICSP" gate="G$1" pin="1"/>
-<wire x1="38.1" y1="73.66" x2="25.4" y2="73.66" width="0.1524" layer="91"/>
-<label x="25.4" y="73.66" size="1.778" layer="95"/>
+<segment>
+<pinref part="IN_EXT1" gate="G$1" pin="3"/>
+<wire x1="215.9" y1="147.32" x2="231.14" y2="147.32" width="0.1524" layer="91"/>
+<label x="231.14" y="147.32" size="1.778" layer="95" rot="MR0"/>
+</segment>
+<segment>
+<pinref part="IN_EXT0" gate="G$1" pin="3"/>
+<wire x1="177.8" y1="147.32" x2="193.04" y2="147.32" width="0.1524" layer="91"/>
+<label x="193.04" y="147.32" size="1.778" layer="95" rot="MR0"/>
 </segment>
 </net>
@@
 </segment>
 <segment>
-<pinref part="AVR_ICSP" gate="G$1" pin="3"/>
-<wire x1="38.1" y1="71.12" x2="25.4" y2="71.12" width="0.1524" layer="91"/>
-<label x="25.4" y="71.12" size="1.778" layer="95"/>
-</segment>
-<segment>
 <pinref part="U$2" gate="G$1" pin="(PCINT1/AIN0/ADC1)PA1"/>
 <wire x1="86.36" y1="99.06" x2="106.68" y2="99.06" width="0.1524" layer="91"/>
@@
 <net name="INPUT_EXT1" class="0">
 <segment>
-<pinref part="IN_EXT1" gate="G$1" pin="3"/>
-<wire x1="215.9" y1="147.32" x2="231.14" y2="147.32" width="0.1524" layer="91"/>
-<label x="231.14" y="147.32" size="1.778" layer="95" rot="MR0"/>
-</segment>
-<segment>
 <pinref part="U$2" gate="G$1" pin="(PCINT3/T0/ADC3)PA3"/>
 <wire x1="86.36" y1="104.14" x2="106.68" y2="104.14" width="0.1524" layer="91"/>
@@
 <label x="142.24" y="88.9" size="1.778" layer="95" rot="MR0"/>
 </segment>
+<segment>
+<wire x1="215.9" y1="144.78" x2="231.14" y2="144.78" width="0.1524" layer="91"/>
+<pinref part="IN_EXT1" gate="G$1" pin="2"/>
+<label x="231.14" y="144.78" size="1.778" layer="95" rot="MR0"/>
+</segment>
 </net>
 <net name="INPUT_EXT0" class="0">
-<segment>
-<pinref part="IN_EXT0" gate="G$1" pin="3"/>
-<wire x1="177.8" y1="147.32" x2="193.04" y2="147.32" width="0.1524" layer="91"/>
-<label x="193.04" y="147.32" size="1.778" layer="95" rot="MR0"/>
-</segment>
 <segment>
 <pinref part="U$2" gate="G$1" pin="(PCINT2/AIN1/ADC2)PA2"/>
@@
 <label x="142.24" y="96.52" size="1.778" layer="95" rot="MR0"/>
 </segment>
+<segment>
+<pinref part="IN_EXT0" gate="G$1" pin="2"/>
+<wire x1="177.8" y1="144.78" x2="193.04" y2="144.78" width="0.1524" layer="91"/>
+<label x="193.04" y="144.78" size="1.778" layer="95" rot="MR0"/>
+</segment>
 </net>
 <net name="PWM0" class="0">
@@
 <label x="106.68" y="111.76" size="1.778" layer="95" rot="MR0"/>
 </segment>
-</net>
-<net name="PWM1" class="0">
 <segment>
 <pinref part="AVR_ICSP" gate="G$1" pin="4"/>
@@
 <label x="63.5" y="71.12" size="1.778" layer="95"/>
 </segment>
+</net>
+<net name="PWM1" class="0">
 <segment>
 <pinref part="PWM1A" gate="G$1" pin="1"/>
@@
 <wire x1="86.36" y1="109.22" x2="106.68" y2="109.22" width="0.1524" layer="91"/>
 <label x="106.68" y="109.22" size="1.778" layer="95" rot="MR0"/>
+</segment>
+<segment>
+<pinref part="AVR_ICSP" gate="G$1" pin="1"/>
+<wire x1="38.1" y1="73.66" x2="25.4" y2="73.66" width="0.1524" layer="91"/>
+<label x="25.4" y="73.66" size="1.778" layer="95"/>
 </segment>
 </net>
@@
 </segment>
 <segment>
-<pinref part="LED3" gate="G$1" pin="A"/>
+<pinref part="R6" gate="G$1" pin="2"/>
 <wire x1="76.2" y1="40.64" x2="76.2" y2="48.26" width="0.1524" layer="91"/>
 <label x="76.2" y="45.72" size="1.778" layer="95"/>
@@
 </segment>
 <segment>
-<pinref part="LED2" gate="G$1" pin="A"/>
+<pinref part="R5" gate="G$1" pin="2"/>
 <wire x1="60.96" y1="40.64" x2="60.96" y2="48.26" width="0.1524" layer="91"/>
 <label x="60.96" y="45.72" size="1.778" layer="95"/>
@@
 <wire x1="45.72" y1="40.64" x2="45.72" y2="48.26" width="0.1524" layer="91"/>
 <label x="45.72" y="45.72" size="1.778" layer="95"/>
+</segment>
+<segment>
+<pinref part="AVR_ICSP" gate="G$1" pin="3"/>
+<wire x1="38.1" y1="71.12" x2="25.4" y2="71.12" width="0.1524" layer="91"/>
+<label x="25.4" y="71.12" size="1.778" layer="95"/>
 </segment>
 </net>
@@
 <net name="N$2" class="0">
 <segment>
-<pinref part="R5" gate="G$1" pin="2"/>
-<pinref part="LED2" gate="G$1" pin="C"/>
-<wire x1="60.96" y1="30.48" x2="60.96" y2="33.02" width="0.1524" layer="91"/>
+<pinref part="R5" gate="G$1" pin="1"/>
+<pinref part="LED2" gate="G$1" pin="A"/>
+<wire x1="60.96" y1="30.48" x2="60.96" y2="27.94" width="0.1524" layer="91"/>
 </segment>
 </net>
 <net name="N$5" class="0">
 <segment>
-<pinref part="R6" gate="G$1" pin="2"/>
-<pinref part="LED3" gate="G$1" pin="C"/>
-<wire x1="76.2" y1="30.48" x2="76.2" y2="33.02" width="0.1524" layer="91"/>
-</segment>
-</net>
+<pinref part="LED3" gate="G$1" pin="A"/>
+<pinref part="R6" gate="G$1" pin="1"/>
+<wire x1="76.2" y1="27.94" x2="76.2" y2="30.48" width="0.1524" layer="91"/>
+</segment>
+</net>

Commit message: Updates to rev4.
Parts:
- removed AVR_ICSP: AVR_SPI_PRG_6PTH, SparkFun-Connectors:AVR_SPI_PRG_6PTH
- removed C4: 22uF 10V, SparkFun-Capacitors:CAP_POL1206
- removed IN_EXT1: (no value), SparkFun-Connectors:M03PTH
- removed JP1: M02PTH, SparkFun-Connectors:M02PTH
- removed POT1: (no value), SparkFun-Electromechanical:POT
- removed STANDOFF2: STAND-OFF, SparkFun-Electromechanical:STAND-OFF
- added C2: 22uF 10V, SparkFun-Capacitors:CAP1206
- added JP2: M01PTH, SparkFun-Connectors:M01PTH
- added R7: 10K, SparkFun-Resistors:RESISTOR0603
- added R8: 100K, SparkFun-Resistors:RESISTOR0603
- added STEER, SW, THR, THR1: (no value), SparkFun-Connectors:M03PTH
- added U$3: JSH-GH-2VERT, BlueRobotics-JST-GH:JSH-GH-2VERT
- R1, R2: value 1M -> 100K
- U$1: value LOGOFULL-M -> LOGOBR-LOGO-MS; device BlueRobotics-Main:LOGOFULL-M -> BlueRobotics-Main:LOGOBR-LOGO-MS
- renumbered IN_EXT0 to THR0
Connections:
- net INPUT_EXT0 renamed THROTTLE0
- removed net INPUT_EXT1: IN_EXT1.2, R2.2, U$2.(PCINT3/T0/ADC3)PA3
- removed net INPUT_INT: POT1.S, U$2.(PCINT1/AIN0/ADC1)PA1
- removed net LED_INT: AVR_ICSP.3, LED1.A, U$2.(PCINT4/T1/SCL/USCK/ADC4)PA4
- new net STEERING: R8.2, STEER.2, U$2.(PCINT1/AIN0/ADC1)PA1
- new net SWITCH: R7.1, SW.2, U$2.(PCINT4/T1/SCL/USCK/ADC4)PA4
- new net THROTTLE1: R2.2, THR.2, THR1.2, U$2.(PCINT3/T0/ADC3)PA3
- net +5V: now also C2.1, LED1.A, R7.2, STEER.3, SW.3, THR.3, THR1.3; no longer AVR_ICSP.2, C4.+, IN_EXT1.3, POT1.E
- net DETECT: now also R8.1
- net GND: now also C2.2, STEER.1, SW.1, THR.1, THR1.1, U$3.2; no longer AVR_ICSP.6, C4.-, IN_EXT1.1, JP1.1, POT1.A
- net PWM0: now also U$2.(PCINT5/OC1B/MISO/DO/ADC5)PA5; no longer AVR_ICSP.4, U$2.(PCINT6/OC1A/SDA/MOSI/ADC6)PA6
- net PWM1: now also U$2.(PCINT6/OC1A/SDA/MOSI/ADC6)PA6; no longer AVR_ICSP.1, U$2.(PCINT5/OC1B/MISO/DO/ADC5)PA5
- net RESET: now also JP2.1; no longer AVR_ICSP.5
- net VIN: now also U$3.1; no longer JP1.2
Other:
- note added: "AVR ISP HERE"
