File: Hardware/Thruster-Commander-Programmer.sch (EAGLE design)
At the start: 12 parts, among them J1 AVR_SPI_PROG_3X2PTH

Commit message: Fix programmer board MISO/MOSI connections
Parts:
- renumbered PWM0A to PWM_L_A, PWM0B to PWM_L_B, PWM1A to PWM_R_A, PWM1B to PWM_R_B
Connections:
- removed net PWM0: J1.4, PWM_L_A.1, PWM_L_B.1
- removed net PWM1: J1.1, PWM_R_A.1, PWM_R_B.1
- new net PWM_L: J1.1, PWM_L_A.1, PWM_L_B.1
- new net PWM_R: J1.4, PWM_R_A.1, PWM_R_B.1
- net +5V: now also PWM_L_B.2
Changed lines of the file:
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@@
 </classes>
 <parts>
-<part name="PWM0A" library="SparkFun-Connectors" deviceset="M03" device="PTH"/>
-<part name="PWM0B" library="SparkFun-Connectors" deviceset="M03" device="PTH"/>
-<part name="PWM1A" library="SparkFun-Connectors" deviceset="M03" device="PTH"/>
-<part name="PWM1B" library="SparkFun-Connectors" deviceset="M03" device="PTH"/>
+<part name="PWM_L_A" library="SparkFun-Connectors" deviceset="M03" device="PTH"/>
+<part name="PWM_L_B" library="SparkFun-Connectors" deviceset="M03" device="PTH"/>
+<part name="PWM_R_A" library="SparkFun-Connectors" deviceset="M03" device="PTH"/>
+<part name="PWM_R_B" library="SparkFun-Connectors" deviceset="M03" device="PTH"/>
 <part name="THR0" library="SparkFun-Connectors" deviceset="M03" device="PTH"/>
 <part name="THR1" library="SparkFun-Connectors" deviceset="M03" device="PTH"/>
@@
 </plain>
 <instances>
-<instance part="PWM0A" gate="G$1" x="114.3" y="55.88"/>
-<instance part="PWM0B" gate="G$1" x="147.32" y="55.88"/>
-<instance part="PWM1A" gate="G$1" x="182.88" y="55.88"/>
-<instance part="PWM1B" gate="G$1" x="215.9" y="55.88"/>
+<instance part="PWM_L_A" gate="G$1" x="114.3" y="55.88"/>
+<instance part="PWM_L_B" gate="G$1" x="147.32" y="55.88"/>
+<instance part="PWM_R_A" gate="G$1" x="182.88" y="55.88"/>
+<instance part="PWM_R_B" gate="G$1" x="215.9" y="55.88"/>
 <instance part="THR0" gate="G$1" x="170.18" y="144.78"/>
 <instance part="THR1" gate="G$1" x="170.18" y="127"/>
@@
 </segment>
 <segment>
-<pinref part="PWM0A" gate="G$1" pin="2"/>
+<pinref part="PWM_L_A" gate="G$1" pin="2"/>
 <wire x1="121.92" y1="55.88" x2="129.54" y2="55.88" width="0.1524" layer="91"/>
 <label x="129.54" y="55.88" size="1.778" layer="95" rot="MR0"/>
+</segment>
+<segment>
+<pinref part="PWM_L_B" gate="G$1" pin="2"/>
+<wire x1="154.94" y1="55.88" x2="162.56" y2="55.88" width="0.1524" layer="91"/>
+<label x="162.56" y="55.88" size="1.778" layer="95" rot="MR0"/>
 </segment>
 </net>
@@
 </segment>
 </net>
-<net name="PWM0" class="0">
-<segment>
-<pinref part="PWM0A" gate="G$1" pin="1"/>
-<wire x1="121.92" y1="53.34" x2="129.54" y2="53.34" width="0.1524" layer="91"/>
-<label x="124.46" y="53.34" size="1.778" layer="95"/>
-</segment>
-<segment>
-<pinref part="PWM0B" gate="G$1" pin="1"/>
-<wire x1="154.94" y1="53.34" x2="160.02" y2="53.34" width="0.1524" layer="91"/>
-<label x="157.48" y="53.34" size="1.778" layer="95"/>
-</segment>
-<segment>
-<wire x1="55.88" y1="71.12" x2="68.58" y2="71.12" width="0.1524" layer="91"/>
-<label x="63.5" y="71.12" size="1.778" layer="95"/>
-<pinref part="J1" gate="G$1" pin="4"/>
-</segment>
-</net>
-<net name="PWM1" class="0">
-<segment>
-<pinref part="PWM1A" gate="G$1" pin="1"/>
-<wire x1="190.5" y1="53.34" x2="195.58" y2="53.34" width="0.1524" layer="91"/>
-<label x="193.04" y="53.34" size="1.778" layer="95"/>
-</segment>
-<segment>
-<pinref part="PWM1B" gate="G$1" pin="1"/>
-<wire x1="223.52" y1="53.34" x2="228.6" y2="53.34" width="0.1524" layer="91"/>
-<label x="226.06" y="53.34" size="1.778" layer="95"/>
-</segment>
-<segment>
-<wire x1="38.1" y1="73.66" x2="25.4" y2="73.66" width="0.1524" layer="91"/>
-<label x="25.4" y="73.66" size="1.778" layer="95"/>
-<pinref part="J1" gate="G$1" pin="1"/>
-</segment>
-</net>
 <net name="SWITCH" class="0">
 <segment>
@@
 </segment>
 </net>
+<net name="PWM_L" class="0">
+<segment>
+<pinref part="PWM_L_A" gate="G$1" pin="1"/>
+<wire x1="121.92" y1="53.34" x2="129.54" y2="53.34" width="0.1524" layer="91"/>
+<label x="124.46" y="53.34" size="1.778" layer="95"/>
+</segment>
+<segment>
+<pinref part="PWM_L_B" gate="G$1" pin="1"/>
+<wire x1="154.94" y1="53.34" x2="162.56" y2="53.34" width="0.1524" layer="91"/>
+<label x="157.48" y="53.34" size="1.778" layer="95"/>
+</segment>
+<segment>
+<wire x1="38.1" y1="73.66" x2="25.4" y2="73.66" width="0.1524" layer="91"/>
+<label x="25.4" y="73.66" size="1.778" layer="95"/>
+<pinref part="J1" gate="G$1" pin="1"/>
+</segment>
+</net>
+<net name="PWM_R" class="0">
+<segment>
+<pinref part="PWM_R_A" gate="G$1" pin="1"/>
+<wire x1="190.5" y1="53.34" x2="195.58" y2="53.34" width="0.1524" layer="91"/>
+<label x="193.04" y="53.34" size="1.778" layer="95"/>
+</segment>
+<segment>
+<pinref part="PWM_R_B" gate="G$1" pin="1"/>
+<wire x1="223.52" y1="53.34" x2="228.6" y2="53.34" width="0.1524" layer="91"/>
+<label x="226.06" y="53.34" size="1.778" layer="95"/>
+</segment>
+<segment>
+<wire x1="55.88" y1="71.12" x2="68.58" y2="71.12" width="0.1524" layer="91"/>
+<label x="63.5" y="71.12" size="1.778" layer="95"/>
+<pinref part="J1" gate="G$1" pin="4"/>
+</segment>
+</net>
